File: HW/GreenFox/GreenFox.kicad_pcb (KiCad board)
At the start: 2 copper layers, 20.3 x 46.4 mm, 29 parts, among them J1 USB_C_Receptacle_USB2.0, J2 Conn_02x05_Odd_Even, J3 Conn_01x14, J5 Conn_01x14, SW1 SW_Push, SW2 SW_Push, U1 LN1134-3.3V, U2 SRV05-4, U3 PIC32MM0256GPM036-IM2, Y1 Crystal_GND2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

Commit message: Finished board, added text, fiducials, logos, etc.
Parts:
- added FID1: Fiducial, Fiducial:Fiducial_0.5mm_Mask1mm, F.Cu at (124.5, 64.6)
- added FID2: Fiducial, Fiducial:Fiducial_0.5mm_Mask1mm, F.Cu at (116.2, 106.0)
- added FID3: Fiducial, Fiducial:Fiducial_0.5mm_Mask1mm, F.Cu at (132.7, 106.0)
- added MARK1: LOGO, KiCAD library:FOX_LOGO_MASK, B.Cu at (124.5, 72.0)
- added MARK2: Logo_Open_Hardware_Small, Symbol:OSHW-Logo_7.5x8mm_SilkScreen, B.Cu at (124.5, 92.9)
- Y1: value Crystal_GND2 -> 8MHz
- Y2: value Crystal -> 32.768kHz
- moved C3 0.25 mm to (128.0, 88.5)
- moved D3 0.23 mm to (123.2, 90.0)
- moved R9 0.23 mm to (119.8, 90.0)
- moved D2 0.19 mm to (123.2, 88.6)
- moved R8 0.19 mm to (119.8, 88.6)
- moved C7 0.06 mm to (128.0, 74.9)
Routing:
- net GND: track 31.3 -> 37.6 mm, vias 25 -> 103
- net /UART1_RX: track 39.2 -> 41.1 mm
- net /LED_USER: track 33.1 -> 31.4 mm
- net /TCK: track 37.4 -> 38.5 mm
- net /SOSCO: track 7.27 -> 7.78 mm
- net +3V3: track 84.4 -> 84.2 mm, vias 8 -> 7
Other:
- board text added: "3V"
- board text added: "5V"
- board text added: "A0"
- board text added: "A1"
- board text added: "A9"
- board text added: "B0"
- board text added: "B1"
- board text added: "B10"
- board text added: "B11"
- board text added: "B13"
- board text added: "B14"
- board text added: "B15"
- board text added: "B2"
- board text added: "B3"
- board text added: "B5"
- board text added: "B7"
- board text added: "B8"
- board text added: "B9"
- board text added: "C0"
- board text added: "C1"
- board text added: "C2"
- board text added: "C8"
- board text added: "C9"
- board text added: "GND"
- board text added: "Green Fox"
- board text added: "Rev1"
- board text added: "~RST~"

Commit message: Minor tweaks, added gerbers
Parts:
- added H1: MB_0.5mm, KiCAD library:MouseBiteHole_0.5mm, F.Cu at (118.5, 101.6)
- added H2: MB_0.5mm, KiCAD library:MouseBiteHole_0.5mm, F.Cu at (120.0, 101.6)
- added H3: MB_0.5mm, KiCAD library:MouseBiteHole_0.5mm, F.Cu at (121.5, 101.6)
- added H4: MB_0.5mm, KiCAD library:MouseBiteHole_0.5mm, F.Cu at (123.0, 101.6)
- added H5: MB_0.5mm, KiCAD library:MouseBiteHole_0.5mm, F.Cu at (124.5, 101.6)
- added H6: MB_0.5mm, KiCAD library:MouseBiteHole_0.5mm, F.Cu at (126.0, 101.6)
- added H7: MB_0.5mm, KiCAD library:MouseBiteHole_0.5mm, F.Cu at (127.5, 101.6)
- added H8: MB_0.5mm, KiCAD library:MouseBiteHole_0.5mm, F.Cu at (129.0, 101.6)
- added H9: MB_0.5mm, KiCAD library:MouseBiteHole_0.5mm, F.Cu at (130.5, 101.6)
Routing:
- net GND: track 37.6 -> 41.9 mm, vias 103 -> 105
- net /TDO\PGEC3: track 42.3 -> 43.4 mm
- net +3V3: track 84.2 -> 85.1 mm
- net /TMS: track 45.9 -> 46.6 mm
- net /UART1_TX: track 42.4 -> 41.8 mm
- net /TDI: track 33.6 -> 34.1 mm
- net /UART1_RX: track 41.1 -> 41.6 mm

Commit message: Add text to buttons and re-export
Other:
- board text added: "RST"
- board text added: "USER"

Commit message: Very quick mod for different fab
Parts:
- removed MARK2: Logo_Open_Hardware_Small, Symbol:OSHW-Logo_7.5x8mm_SilkScreen
- J1: footprint KiCAD library:Jing USB C 2.0 16pin receptable -> Neofoxx's Library:Jing_USB_C_2_0_16pin_receptable_noSlots
- moved R2 2.68 mm to (129.1, 71.5), turned to 0 degrees
- moved D1 1.88 mm to (118.5, 66.2)
- moved R3 1.14 mm to (130.3, 66.4)
Connections:
- net /~RESET~ renamed /~{RESET}
- J1 pad A8: (no net) -> unconnected-(J1-PadA8)
- J1 pad B8: (no net) -> unconnected-(J1-PadB8)
- U1 pad 4: (no net) -> unconnected-(U1-Pad4)
- U2 pad 4: (no net) -> unconnected-(U2-Pad4)
Routing:
- net GND: track 41.9 -> 37.2 mm, vias 105 -> 102
- net Net-(J1-PadA5): track 8.74 -> 11.1 mm
- net Net-(D1-Pad2): track 13.1 -> 14.4 mm
- net Net-(J1-PadB5): track 10.5 -> 11.6 mm
- net /RB11: track 11.1 -> 11.9 mm
Other:
- outline, holes or cut-outs redrawn
- net class Default removed
- board text added: "GreenFox Rev1b"
- board text added: "~{RST}"
- board text removed: "Green Fox"
- board text removed: "Rev1"
- board text removed: "~RST~"
